File: relaybrd.kicad_sch (KiCad schematic)
At the start: 16 parts, among them J7 5499922-4, U10 TPS3850H50DRCR

Commit message: Finalize BOM
Parts:
- R44, R45: MFG_PN ERJ-2RKF1001X -> ERJ-2GE0R00X
Changed lines of the file:
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@@
 			)
 		)
-		(property "Description" "RES SMD 1K OHM 1% 1/10W 0402"
+		(property "Description" "RES SMD 0 OHM 1%  0402 JUMPER"
 			(at 172.72 76.2 0)
 			(effects
@@
 			)
 		)
-		(property "MFG_PN" "ERJ-2RKF1001X"
+		(property "MFG_PN" "ERJ-2GE0R00X"
 			(at 172.72 76.2 0)
 			(effects
@@
 			)
 		)
-		(property "Description" "RES SMD 1K OHM 1% 1/10W 0402"
+		(property "Description" "RES SMD 0 OHM 1%  0402 JUMPER"
 			(at 172.72 85.09 0)
 			(effects
@@
 			)
 		)
-		(property "MFG_PN" "ERJ-2RKF1001X"
+		(property "MFG_PN" "ERJ-2GE0R00X"
 			(at 172.72 85.09 0)
 			(effects
